File: GF24.kicad_sch (KiCad schematic)
At the start: 67 parts, among them J1 USB4110GFA, J3 Conn_ARM_SWD_TagConnect_TC2030, J4 Conn_01x04_Pin, Q1 3904, SW1 EG1205, SW3 BOOT, SW4 EG1205, SW5 360-2674-ND, U1 TPS79533DCQR, U2 LTC1733, U3 SAM-M10Q, U4 STM32F102C8Tx, X1 ECS-2520MV-160-CN

Commit message: updated BOM, ordered board/components
Parts:
- SW1, SW4: Manufacturer PN (none) -> EG1205-ND
- SW5: Manufacturer PN (none) -> 360-2674-ND
Changed lines of the file:
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@@
 	(label "CH-PROG"
 		(at 73.66 40.64 0)
-		(fields_autoplaced yes)
 		(effects
 			(font
@@
 	(label "USBC+"
 		(at 138.43 17.78 0)
-		(fields_autoplaced yes)
 		(effects
 			(font
@@
 	(label "Noise_Reduction"
 		(at 196.85 29.21 0)
-		(fields_autoplaced yes)
 		(effects
 			(font
@@
 	(label "BACKUP_DEBUG_ST_RX"
 		(at 114.3 116.84 0)
-		(fields_autoplaced yes)
 		(effects
 			(font
@@
 	(label "BUZZ-QB"
 		(at 246.38 153.67 270)
-		(fields_autoplaced yes)
 		(effects
 			(font
@@
 	(label "SWDCLK"
 		(at 139.7 127 0)
-		(fields_autoplaced yes)
 		(effects
 			(font
@@
 	(label "REG_I"
 		(at 170.18 21.59 0)
-		(fields_autoplaced yes)
 		(effects
 			(font
@@
 	(label "CH-TIMER"
 		(at 63.5 38.1 0)
-		(fields_autoplaced yes)
 		(effects
 			(font
@@
 	(label "CLK_OUT"
 		(at 46.99 111.76 0)
-		(fields_autoplaced yes)
 		(effects
 			(font
@@
 	(label "BOOT0_RES"
 		(at 49.53 90.17 0)
-		(fields_autoplaced yes)
 		(effects
 			(font
@@
 	(label "ACT-H"
 		(at 259.08 82.55 180)
-		(fields_autoplaced yes)
 		(effects
 			(font
@@
 	(label "BAT+"
 		(at 113.03 30.48 0)
-		(fields_autoplaced yes)
 		(effects
 			(font
@@
 	(label "MODE-H"
 		(at 223.52 82.55 0)
-		(fields_autoplaced yes)
 		(effects
 			(font
@@
 	(label "SWDIO"
 		(at 139.7 124.46 0)
-		(fields_autoplaced yes)
 		(effects
 			(font
@@
 	(label "BACKUP_DEBUG_ST_TX"
 		(at 114.3 114.3 0)
-		(fields_autoplaced yes)
 		(effects
 			(font
@@
 	(label "BUZZ-"
 		(at 260.35 146.05 0)
-		(fields_autoplaced yes)
 		(effects
 			(font
@@
 	(label "BOOT0_I"
 		(at 67.31 90.17 0)
-		(fields_autoplaced yes)
 		(effects
 			(font
@@
 	(label "CH-TH-DIV"
 		(at 55.88 35.56 0)
-		(fields_autoplaced yes)
 		(effects
 			(font
@@
 	(label "DEBUG_ST_RX"
 		(at 58.42 147.32 0)
-		(fields_autoplaced yes)
 		(effects
 			(font
@@
 	(label "DEBUG_ST_TX"
 		(at 58.42 144.78 0)
-		(fields_autoplaced yes)
 		(effects
 			(font
@@
 			)
 		)
+		(property "Manufacturer PN" "EG1205-ND"
+			(at 161.29 21.59 0)
+			(effects
+				(font
+					(size 1.27 1.27)
+				)
+				(hide yes)
+			)
+		)
 		(pin "2"
 		)
@@
 			)
 		)
+		(property "Manufacturer PN" "360-2674-ND"
+			(at 259.08 92.71 0)
+			(effects
+				(font
+					(size 1.27 1.27)
+				)
+				(hide yes)
+			)
+		)
 		(pin "2"
 		)
@@
 			(at 223.52 90.17 0)
 			(effects
+				(font
+					(size 1.27 1.27)
+				)
+				(hide yes)
+			)
+		)
+		(property "Manufacturer PN" "EG1205-ND"
+			(at 223.52 90.17 0)
+			(effects
